File: beeb_wifiport.kicad_pcb (KiCad board)
At the start: 2 copper layers, 28 x 28 mm, 18 parts, among them J1 User Port, J2 USB4105-GF-A, J3 1040310811, SW1 EVQ-P7A01P, SW2 EVQ-P7A01P, U1 ESP32-S3-MINI-1, U3 LDL212PV33R, U4 NXB0104GU12

Commit message: Clarify part numbers
Parts:
- D1: value PMEG2020CPA -> PMEG2020CPA,115
- J1: value User Port -> 613020243121
- U1: value ESP32-S3-MINI-1 -> ESP32-S3-MINI-1-N4R2
Changed lines of the file:
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@@
 			)
 		)
-		(property "Value" "ESP32-S3-MINI-1"
+		(property "Value" "ESP32-S3-MINI-1-N4R2"
 			(at 0 3.55 0)
 			(unlocked yes)
@@
 			)
 		)
-		(property "Value" "PMEG2020CPA"
+		(property "Value" "PMEG2020CPA,115"
 			(at 0 1.95 0)
 			(layer "F.Fab")
@@
 			)
 		)
-		(property "Value" "User Port"
+		(property "Value" "613020243121"
 			(at -5.65 25.63 90)
 			(layer "F.Fab")
